File: kicad-import/adafruit-ethernet/Adafruit Ethernet FeatherWing.kicad_sch (KiCad schematic)
At the start: 44 parts, among them IC2 74AHC1G125, U2 W5500, X3 RB1-125BAG1A, Y1 25MHz

Commit message: Initial sheet settings for layout.
Other:
- company: (none) -> Kingdom Metrics
- title: (none) -> Genesis Board
Changed lines of the file:
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@@
 	(generator_version "9.0")
 	(paper "User" 303.962 217.322)
+	(title_block
+		(title "Genesis Board")
+		(date "2025-05-27")
+		(rev "0.1")
+		(company "Kingdom Metrics")
+	)
 	(text "Internal pullup on CS"
 		(exclude_from_sim no)
