File: rev1/Genesis/Genesis.kicad_pcb (KiCad board)
At the start: 2 copper layers, 0 parts

Commit message: Add imported symbol libraries to project
Parts:
- added B1: cr1220, adalogger featherwing:CR1220-2, F.Cu at (-95.6, 15.4)
- added C1: 10µF, Adafruit ESP32 Feather V2:0805-NO, F.Cu at (-75.9, -22.0)
- added C10: 0.1uF, Adafruit ESP32 Feather V2:0603-NO, F.Cu at (-84.0, -11.9)
- added C12: 22pF, Adafruit Ethernet FeatherWing:0603-NO, F.Cu at (-57.6, 8.06)
- added C13: 10uF, Adafruit Ethernet FeatherWing:0805-NO, F.Cu at (-53.0, 25.6)
- added C14: 22pF, Adafruit Ethernet FeatherWing:0603-NO, F.Cu at (-57.6, 10.6)
- added C15: 0.1uF, Adafruit Ethernet FeatherWing:0603-NO, F.Cu at (-57.6, 13.1)
- added C16: 0.1uF, Adafruit Ethernet FeatherWing:0603-NO, F.Cu at (-57.6, 15.6)
- added C17: 10uF, Adafruit Ethernet FeatherWing:0805-NO, F.Cu at (-53.0, 28.1)
- added C18: 0.1uF, Adafruit Ethernet FeatherWing:0603-NO, F.Cu at (-57.6, 18.1)
- added C19: 0.1uF, Adafruit Ethernet FeatherWing:0603-NO, F.Cu at (-57.6, 20.6)
- added C2: 10µF, Adafruit ESP32 Feather V2:0805-NO, F.Cu at (-75.9, -19.5)
- added C20: 0.1uF, Adafruit Ethernet FeatherWing:0603-NO, F.Cu at (-57.6, 23.1)
- added C21: 0.1uF, Adafruit Ethernet FeatherWing:0603-NO, F.Cu at (-53.6, 8.06)
- added C22: 10uF, Adafruit Ethernet FeatherWing:0805-NO, F.Cu at (-53.0, 30.6)
- added C23: 6.8nF, Adafruit Ethernet FeatherWing:0603-NO, F.Cu at (-53.6, 10.6)
- added C24: 10nF, Adafruit Ethernet FeatherWing:0603-NO, F.Cu at (-53.6, 13.1)
- added C25: 10nF, Adafruit Ethernet FeatherWing:0603-NO, F.Cu at (-53.6, 15.6)
- added C26: 6.8nF, Adafruit Ethernet FeatherWing:0603-NO, F.Cu at (-53.6, 18.1)
- added C27: 10uF, adalogger featherwing:0805-NO, F.Cu at (-83.6, 39.8)
- added C28: 10uF, adalogger featherwing:0805-NO, F.Cu at (-83.6, 42.3)
- added C3: 10uF, Adafruit ESP32 Feather V2:0805-NO, F.Cu at (-75.9, -17.0)
- added C4: 1uF, Adafruit ESP32 Feather V2:0603-NO, F.Cu at (-84.0, -22.0)
- added C5: 10uF, Adafruit ESP32 Feather V2:0805-NO, F.Cu at (-75.9, -14.5)
- added C6: 10uF, Adafruit ESP32 Feather V2:0805-NO, F.Cu at (-75.9, -12.0)
- added C7: 1uF, Adafruit ESP32 Feather V2:0603-NO, F.Cu at (-84.0, -19.4)
- added C8: 0.1uF, Adafruit ESP32 Feather V2:0603-NO, F.Cu at (-84.0, -16.9)
- added C9: 1uF, Adafruit ESP32 Feather V2:0603-NO, F.Cu at (-84.0, -14.4)
- added D1: MBR540, Adafruit ESP32 Feather V2:SOD-123, F.Cu at (-70.8, -13.4)
- added D2: RED, Adafruit ESP32 Feather V2:CHIPLED_0603_NOOUTLINE, F.Cu at (-94.3, -3.41)
- added FB1: ferrite, Adafruit Ethernet FeatherWing:0805-NO, F.Cu at (-53.0, 33.1)
- added FB2: ferrite, Adafruit Ethernet FeatherWing:0805-NO, F.Cu at (-53.0, 35.6)
- added FID1: FIDUCIAL"", Adafruit Ethernet FeatherWing:FIDUCIAL_1MM, F.Cu at (-66.6, 31.9)
- added FID2: FIDUCIAL"", Adafruit Ethernet FeatherWing:FIDUCIAL_1MM, F.Cu at (-66.6, 34.9)
- added FID3: FIDUCIAL"", Adafruit Ethernet FeatherWing:FIDUCIAL_1MM, F.Cu at (-66.6, 37.9)
- added FID4: FIDUCIAL_1MM, adalogger featherwing:FIDUCIAL_1MM, F.Cu at (-83.3, 18.3)
- added FID5: FIDUCIAL_1MM, adalogger featherwing:FIDUCIAL_1MM, F.Cu at (-83.3, 21.3)
- added IC1: CP2102N-24, Adafruit ESP32 Feather V2:QFN24_4MM_SMSC, F.Cu at (-83.1, 1.21)
- added IC2: 74AHC1G125, Adafruit Ethernet FeatherWing:SOT23-5L, F.Cu at (-49.0, 34.2)
- added IC3: PCF8523T, adalogger featherwing:SOIC8_150MIL, F.Cu at (-87.1, 34.3)
- added INT1: HEADER-1X1ROUND, adalogger featherwing:1X01_ROUND, F.Cu at (-82.8, 31.4)
- added JP1: HEADER-1X12, Adafruit ESP32 Feather V2:1X12_ROUND, F.Cu at (-89.9, -24.5)
- added JP2: HEADER-1X16ROUND, Adafruit ESP32 Feather V2:1X16_ROUND, F.Cu at (-84.8, -27.2)
- added JP5: HEADER-1X376MIL, Adafruit Ethernet FeatherWing:1X03_ROUND_76, F.Cu at (-46.5, 25.8)
- added LED1: WS2812B3535, Adafruit ESP32 Feather V2:LED3535, F.Cu at (-98.0, -2.59)
- added Q1: DUAL NPN, Adafruit ESP32 Feather V2:SOT363, F.Cu at (-67.9, -9.02)
- added Q2: DUAL NPN, Adafruit ESP32 Feather V2:SOT363, F.Cu at (-67.9, -5.72)
- added R1: 100K, Adafruit ESP32 Feather V2:0603-NO, F.Cu at (-80.0, -22.0)
- added R10: 47K, Adafruit ESP32 Feather V2:RESPACK_4X0603, F.Cu at (-103.2, -5.20)
- added R11: 47K, Adafruit ESP32 Feather V2:RESPACK_4X0603, F.Cu at (-103.2, -1.19)
- added R12: 47K, Adafruit ESP32 Feather V2:RESPACK_4X0603, F.Cu at (-103.2, 2.81)
- added R14: 1M, Adafruit Ethernet FeatherWing:0603-NO, F.Cu at (-53.6, 20.6)
- added R15: 10K, Adafruit Ethernet FeatherWing:0603-NO, F.Cu at (-53.6, 23.1)
- added R16: 470, Adafruit Ethernet FeatherWing:0603-NO, F.Cu at (-49.6, 8.06)
- added R17: 470, Adafruit Ethernet FeatherWing:0603-NO, F.Cu at (-49.6, 10.6)
- added R18: 10K, Adafruit Ethernet FeatherWing:0603-NO, F.Cu at (-49.6, 13.1)
- added R19: 10K, Adafruit Ethernet FeatherWing:0603-NO, F.Cu at (-49.6, 15.6)
- added R2: 47K, Adafruit ESP32 Feather V2:RESPACK_4X0603, F.Cu at (-103.2, -21.2)
- added R20: 10K, Adafruit Ethernet FeatherWing:0603-NO, F.Cu at (-49.6, 18.1)
- added R21: 10K, Adafruit Ethernet FeatherWing:0603-NO, F.Cu at (-49.6, 20.6)
- added R22: 12.4K, Adafruit Ethernet FeatherWing:0603-NO, F.Cu at (-49.6, 23.1)
- added R23: 49.9, Adafruit Ethernet FeatherWing:0603-NO, F.Cu at (-45.6, 8.06)
- added R24: 49.9, Adafruit Ethernet FeatherWing:0603-NO, F.Cu at (-45.6, 10.6)
- added R25: 49.9, Adafruit Ethernet FeatherWing:0603-NO, F.Cu at (-45.6, 13.1)
- added R26: 49.9, Adafruit Ethernet FeatherWing:0603-NO, F.Cu at (-45.6, 15.6)
- added R27: 10, Adafruit Ethernet FeatherWing:0603-NO, F.Cu at (-45.6, 18.1)
- added R28: 10K, Adafruit Ethernet FeatherWing:0603-NO, F.Cu at (-45.6, 20.6)
- added R29: 1K, adalogger featherwing:0603-NO, F.Cu at (-82.8, 8.06)
- added R3: 100K, Adafruit ESP32 Feather V2:0603-NO, F.Cu at (-80.0, -19.4)
- added R30: 100K, adalogger featherwing:0603-NO, F.Cu at (-82.8, 10.6)
- added R31: 10K, adalogger featherwing:0603-NO, F.Cu at (-82.8, 13.1)
- added R32: 10K, adalogger featherwing:0603-NO, F.Cu at (-82.8, 15.6)
- added R4: 10K, Adafruit ESP32 Feather V2:RESPACK_4X0603, F.Cu at (-103.2, -17.2)
- added R5: 10K, Adafruit ESP32 Feather V2:RESPACK_4X0603, F.Cu at (-103.2, -13.2)
- added R6: 5.1K, Adafruit ESP32 Feather V2:0603-NO, F.Cu at (-80.0, -16.9)
- added R7: 10K, Adafruit ESP32 Feather V2:RESPACK_4X0603, F.Cu at (-103.2, -9.20)
- added R8: 5.1K, Adafruit ESP32 Feather V2:0603-NO, F.Cu at (-80.0, -14.4)
- added R9: 5.1K, Adafruit ESP32 Feather V2:0603-NO, F.Cu at (-80.0, -11.9)
- added SDCS1: HEADER-1X1ROUND, adalogger featherwing:1X01_ROUND, F.Cu at (-82.8, 34.1)
- added SJ1: SOLDERJUMPERREFLOW_NOPASTE, Adafruit Ethernet FeatherWing:SOLDERJUMPER_REFLOW_NOPASTE, F.Cu at (-57.3, 26.0)
- added SJ2: SOLDERJUMPERREFLOW_NOPASTE, Adafruit Ethernet FeatherWing:SOLDERJUMPER_REFLOW_NOPASTE, F.Cu at (-57.3, 29.2)
- added SJ3: SOLDERJUMPERREFLOW_NOPASTE, Adafruit Ethernet FeatherWing:SOLDERJUMPER_REFLOW_NOPASTE, F.Cu at (-57.3, 32.5)
- added SJ4: SOLDERJUMPERCLOSED, Adafruit Ethernet FeatherWing:SOLDERJUMPER_CLOSEDWIRE, F.Cu at (-57.3, 35.7)
- added SJ5: SOLDERJUMPER_CLOSED, adalogger featherwing:SOLDERJUMPER_CLOSEDWIRE, F.Cu at (-87.9, 40.1)
- added SW1: KMR2, Adafruit ESP32 Feather V2:BTN_KMR2_4.6X2.8, F.Cu at (-70.9, -21.1)
- added SW2: KMR2, Adafruit ESP32 Feather V2:BTN_KMR2_4.6X2.8, F.Cu at (-70.9, -16.8)
- added U$1: FIDUCIAL_1MM, Adafruit ESP32 Feather V2:FIDUCIAL_1MM, F.Cu at (-68.6, -2.57)
- added U$2: FIDUCIAL_1MM, Adafruit ESP32 Feather V2:FIDUCIAL_1MM, F.Cu at (-68.6, 0.43)
- added U$3: MOUNTINGHOLE2.5, Adafruit ESP32 Feather V2:MOUNTINGHOLE_2.5_PLATED, F.Cu at (-72.7, -8.07)
- added U$4: MOUNTINGHOLE2.5, Adafruit ESP32 Feather V2:MOUNTINGHOLE_2.5_PLATED, F.Cu at (-72.7, -2.87)
- added U1: AP2112-3.3, Adafruit ESP32 Feather V2:SOT23-5, F.Cu at (-98.5, 2.27)
- added U2: W5500, Adafruit Ethernet FeatherWing:LQFP48, F.Cu at (-73.4, 35.7)
- added X1: ESP32-PICO-MINI-02MINI, Adafruit ESP32 Feather V2:ESP32-PICO-MINI, F.Cu at (-93.4, -11.4)
- added X2: USB Type C, Adafruit ESP32 Feather V2:USB_C_CUSB31-CFM2AX-01-X, F.Cu at (-80.7, -6.05)
- added X3: RB1-125BAG1A, Adafruit Ethernet FeatherWing:RJ45_PULSEJACK, F.Cu at (-69.2, 19.0)
- added X4: microsd, adalogger featherwing:MICROSD, F.Cu at (-104.9, 24.8)
- added Y1: 25MHz, Adafruit Ethernet FeatherWing:CRYSTAL_3.2X2.5, F.Cu at (-48.3, 29.6)
- added Y2: 32khz, adalogger featherwing:CRYSTAL_8X3.8, F.Cu at (-85.4, 27.1)

Commit message: Do rough major component placement for layout
Parts:
- moved U$3 330.4 mm to (255.0, 34.0)
- moved U$4 330.4 mm to (255.0, 39.2)
- moved R10 324.7 mm to (193.9, 125.7)
- moved R11 324.7 mm to (193.9, 129.7)
- moved R12 324.7 mm to (193.9, 133.7)
- moved R4 324.7 mm to (193.9, 113.6)
- moved R5 324.7 mm to (193.9, 117.7)
- moved R7 324.7 mm to (193.9, 121.7)
- moved R2 324.3 mm to (193.9, 108.8)
- moved FID4 319.7 mm to (236.0, 34.0)
- moved FID5 319.7 mm to (236.0, 37.0)
- moved U$1 310.1 mm to (240.0, 27.5)
- moved U$2 308.2 mm to (236.5, 43.5)
- moved FID1 304.6 mm to (237.5, 48.5)
- moved FID2 304.6 mm to (237.5, 51.5)
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